Commit message: Update my_robot.xacro

File: my_robot/urdf/my_robot.xacro (robot description, xacro)
@@ -149,5 +149,13 @@
     <dynamics damping="1.0" friction="1.0"/>
   </joint>
-  <!-- Hokuyo Lidar -->
+  <!-- Sensor Upgrade-->
+  <joint name="camera_optical_joint" type="fixed">
+    <origin xyz="0 0 0" rpy="-1.5707 0 -1.5707"/>
+    <parent link="camera_link"/>
+    <child link="camera_link_optical"/>
+  </joint>
+  <link name="camera_link_optical">
+  </link>
+<!-- Hokuyo Lidar -->
   <link name="hokuyo">
     <inertial>

Commit message: Update my_robot.xacro

File: my_robot/urdf/my_robot.xacro (robot description, xacro)
@@ -149,13 +149,5 @@
     <dynamics damping="1.0" friction="1.0"/>
   </joint>
-  <!-- Sensor Upgrade-->
-  <joint name="camera_optical_joint" type="fixed">
-    <origin xyz="0 0 0" rpy="-1.5707 0 -1.5707"/>
-    <parent link="camera_link"/>
-    <child link="camera_link_optical"/>
-  </joint>
-  <link name="camera_link_optical">
-  </link>
-<!-- Hokuyo Lidar -->
+  <!-- Hokuyo Lidar -->
   <link name="hokuyo">
     <inertial>

Commit message: Update my_robot.xacro

File: my_robot/urdf/my_robot.xacro (robot description, xacro)
@@ -149,4 +149,12 @@
     <dynamics damping="1.0" friction="1.0"/>
   </joint>
+  <!-- Upgraded RGB-D camera -->
+  <joint name="camera_optical_joint" type="fixed">
+    <origin xyz="0 0 0" rpy="-1.5707 0 -1.5707"/>
+    <parent link="camera_link"/>
+    <child link="camera_link_optical"/>
+  </joint>
+  <link name="camera_link_optical">
+  </link>
   <!-- Hokuyo Lidar -->
   <link name="hokuyo">

Commit message: Add files via upload

File: my_robot/urdf/my_robot.xacro (robot description, xacro)
@@ -14,7 +14,7 @@
       <origin xyz="0.0 0 0" rpy=" 0 0 0"/>
       <inertia
-          ixx="0.1" ixy="0" ixz="0"
-          iyy="0.1" iyz="0"
-          izz="0.1"
+              ixx="0.1" ixy="0" ixz="0"
+              iyy="0.1" iyz="0"
+              izz="0.1"
       />
     </inertial>
@@ -22,5 +22,5 @@
       <origin xyz="0 0 0" rpy=" 0 0 0"/>
       <geometry>
-        <box size=".4 .2 .088"/>
+        <box size=".4 .2 .1"/>
       </geometry>
     </collision>
@@ -28,5 +28,5 @@
       <origin xyz="0 0 0" rpy=" 0 0 0"/>
       <geometry>
-        <box size=".4 .2 .15"/>
+        <box size=".4 .2 .1"/>
       </geometry>
     </visual>
@@ -56,5 +56,5 @@
     </visual>
   </link>
-  <!-- Robot's two wheels -->
+  <!-- Add two wheels -->
   <link name="left_wheel">
     <inertial>
@@ -69,5 +69,5 @@
       <origin xyz="0 0 0" rpy="0 1.5707 1.5707"/>
       <geometry>
-        <cylinder radius="0.1001" length="0.05"/>
+        <cylinder radius="0.1" length="0.05"/>
       </geometry>
     </collision>
@@ -75,5 +75,5 @@
       <origin xyz="0 0 0" rpy="0 1.5707 1.5707"/>
       <geometry>
-        <cylinder radius="0.1001" length="0.05"/>
+        <cylinder radius="0.1" length="0.05"/>
       </geometry>
     </visual>
@@ -91,5 +91,5 @@
       <origin xyz="0 0 0" rpy="0 1.5707 1.5707"/>
       <geometry>
-        <cylinder radius="0.1001" length="0.05"/>
+        <cylinder radius="0.1" length="0.05"/>
       </geometry>
     </collision>
@@ -97,11 +97,10 @@
       <origin xyz="0 0 0" rpy="0 1.5707 1.5707"/>
       <geometry>
-        <cylinder radius="0.1001" length="0.05"/>
+        <cylinder radius="0.1" length="0.05"/>
       </geometry>
     </visual>
   </link>
-  <!-- Robot's joints for wheels -->
-  <joint type="continuous" name="left_wheel_hinge">
-    <origin xyz="0 0.15 0" rpy="0 0 0"/>
+  <joint name="left_wheel_hinge" type="continuous">
+    <origin xyz="0 0.125 0" rpy="0 0 0"/>
     <child link="left_wheel"/>
     <parent link="chassis"/>
@@ -110,6 +109,6 @@
     <dynamics damping="1.0" friction="1.0"/>
   </joint>
-  <joint type="continuous" name="right_wheel_hinge">
-    <origin xyz="0 -0.15 0" rpy="0 0 0"/>
+  <joint name="right_wheel_hinge" type="continuous">
+    <origin xyz="0 -0.125 0" rpy="0 0 0"/>
     <child link="right_wheel"/>
     <parent link="chassis"/>
@@ -118,8 +117,8 @@
     <dynamics damping="1.0" friction="1.0"/>
   </joint>
-  <!-- Camera -->
- <link name="camera">
+  <!-- Add camera -->
+  <link name="camera">
+    <origin xyz="0 0 0" rpy="0 0 0" />
     <inertial>
-      <origin xyz="0 0 0" rpy="0 0 0"/>
       <mass value="0.1"/>
       <inertia
@@ -129,5 +128,4 @@
     </inertial>
     <collision>
-      <origin xyz="0 0 0" rpy="0 0 0"/>
       <geometry>
         <box size="0.05 0.05 0.05"/>
@@ -135,5 +133,4 @@
     </collision>
     <visual>
-      <origin xyz="0 0 0" rpy="0 0 0"/>
       <geometry>
         <box size="0.05 0.05 0.05"/>
@@ -141,13 +138,11 @@
     </visual>
   </link>
-  <joint type="fixed" name="camera_joint">
-    <origin xyz="0.2 0.0 0" rpy="0 0 0"/>
-    <child link="camera"/>
+  <joint name="camera_joint" type="fixed">
+    <axis xyz="0 1 0"/>
+    <origin xyz="0.2 0 0" rpy="0 0 0" />
     <parent link="chassis"/>
-    <axis xyz="0 1 0" rpy="0 0 0"/>
-    <limit effort="10000" velocity="1000"/>
-    <dynamics damping="1.0" friction="1.0"/>
+    <child link="camera" />
   </joint>
-  <!-- Upgraded RGB-D camera -->
+  <!-- Add RGB-D camera -->
   <joint name="camera_optical_joint" type="fixed">
     <origin xyz="0 0 0" rpy="-1.5707 0 -1.5707"/>
@@ -157,8 +152,8 @@
   <link name="camera_link_optical">
   </link>
-  <!-- Hokuyo Lidar -->
+  <!-- Add Lidar -->
   <link name="hokuyo">
+    <origin xyz="0 0 0" rpy="0 0 0" />
     <inertial>
-      <origin xyz="0 0 0" rpy="0 0 0"/>
       <mass value="1e-5"/>
       <inertia
@@ -168,11 +163,9 @@
     </inertial>
     <collision>
-      <origin xyz="0 0 0" rpy="0 0 0"/>
       <geometry>
-        <box size="0.1 0.1 0.1"/>
+        <box size=".1 .1 .1"/>
       </geometry>
     </collision>
     <visual>
-      <origin xyz="0 0 0" rpy="0 0 0"/>
       <geometry>
         <mesh filename="package://my_robot/meshes/hokuyo.dae"/>
@@ -180,20 +173,18 @@
     </visual>
   </link>
-  <joint type="fixed" name="hokuyo_joint">
-    <origin xyz="0.15 0 0.1" rpy="0 0 0"/>
-    <child link="hokuyo"/>
+  <joint name="hokuyo_joint" type="fixed">
+    <axis xyz="0 1 0"/>
+    <origin xyz="0.15 0 0.1" rpy="0 0 0" />
     <parent link="chassis"/>
-    <axis xyz="0 1 0" rpy="0 0 0"/>
-    <limit effort="10000" velocity="1000"/>
-    <dynamics damping="1.0" friction="1.0"/>
+    <child link="hokuyo" />
   </joint>
-<!-- Add color to components -->
+  <!-- Color the components -->
   <gazebo reference="chassis">
     <material>Gazebo/Orange</material>
   </gazebo>
-  <gazebo reference="right_wheel">
+  <gazebo reference="left_wheel">
     <material>Gazebo/Green</material>
   </gazebo>
-  <gazebo reference="left_wheel">
+  <gazebo reference="right_wheel">
     <material>Gazebo/Green</material>
   </gazebo>
@@ -201,3 +192,3 @@
     <material>Gazebo/Red</material>
   </gazebo>
-</robot>
+  </robot>
